File: kicad/footswitch.sch (KiCad schematic (older format))
At the start: 72 parts, among them IC1 ATMEGA328P-A, P1 Atmega right, P2 Atmega top, P3 Programming header, P4 Atmega bottom, P5 Atmega left, P6 Pot hdr, P7 App select, Q1 BSS214NWH6327XTSA1, Q2 BSS214NWH6327XTSA1, SW1 SW_RST, SW10 SW_SPST, SW2 SW_SPST, SW3 SW_SPST, SW4 SW_SPDT, SW5 SW_SPST, SW6 SW_SPST, SW7 SW_SPST, SW8 SW_SPST, SW9 SW_SPST, U1 nRF24L01+, U2 CD4072BM96, U3 CD4072BM96, Y1 Crystal

Commit message: Finish routing; markings and mounting still missing
Connections:
- net 3V3: now also C12.1, C14.1, R5.2, U1.2 (VCC)
- net VCC: no longer C12.1, C14.1, R5.2, U1.2 (VCC)
Changed lines of the file:
@@
 $EndComp
 Text GLabel 4625 6025 1    40   Input ~ 0
-VCC
+3V3
 $Comp
 L C_Small C14
@@
 $Comp
 L VCC #PWR014
-U 1 1 58ED73E8
-P 3200 6325
-F 0 "#PWR014" H 3200 6175 50  0001 C CNN
-F 1 "VCC" V 3200 6525 50  0000 C CNN
-F 2 "" H 3200 6325 50  0000 C CNN
-F 3 "" H 3200 6325 50  0000 C CNN
-	1    3200 6325
-	0    1    1    0
-$EndComp
-$Comp
-L VCC #PWR015
-U 1 1 58ED73E9
-P 2950 5925
-F 0 "#PWR015" H 2950 5775 50  0001 C CNN
-F 1 "VCC" V 2950 6125 50  0000 C CNN
-F 2 "" H 2950 5925 50  0000 C CNN
-F 3 "" H 2950 5925 50  0000 C CNN
-	1    2950 5925
-	0    1    1    0
-$EndComp
-$Comp
-L VCC #PWR016
 U 1 1 58ED73EC
 P 1350 6125
-F 0 "#PWR016" H 1350 5975 50  0001 C CNN
+F 0 "#PWR014" H 1350 5975 50  0001 C CNN
 F 1 "VCC" V 1350 6325 50  0000 C CNN
 F 2 "" H 1350 6125 50  0000 C CNN
@@
 $EndComp
 $Comp
-L PWR_FLAG #FLG017
+L PWR_FLAG #FLG015
 U 1 1 58ED73ED
 P 800 7125
-F 0 "#FLG017" H 800 7220 50  0001 C CNN
+F 0 "#FLG015" H 800 7220 50  0001 C CNN
 F 1 "PWR_FLAG" V 700 7225 50  0000 C CNN
 F 2 "" H 800 7125 50  0000 C CNN
@@
 $EndComp
 $Comp
-L Earth #PWR018
+L Earth #PWR016
 U 1 1 58ED73F1
 P 2000 7125
-F 0 "#PWR018" H 2000 6875 50  0001 C CNN
+F 0 "#PWR016" H 2000 6875 50  0001 C CNN
 F 1 "Earth" H 2000 6975 50  0001 C CNN
 F 2 "" H 2000 7125 50  0000 C CNN
@@
 $EndComp
 $Comp
-L Earth #PWR019
+L Earth #PWR017
 U 1 1 58ED73F2
 P 2000 7525
-F 0 "#PWR019" H 2000 7275 50  0001 C CNN
+F 0 "#PWR017" H 2000 7275 50  0001 C CNN
 F 1 "Earth" H 2000 7375 50  0001 C CNN
 F 2 "" H 2000 7525 50  0000 C CNN
@@
 $EndComp
 $Comp
-L Earth #PWR020
+L Earth #PWR018
 U 1 1 58ED73F4
 P 2000 7325
-F 0 "#PWR020" H 2000 7075 50  0001 C CNN
+F 0 "#PWR018" H 2000 7075 50  0001 C CNN
 F 1 "Earth" H 2000 7175 50  0001 C CNN
 F 2 "" H 2000 7325 50  0000 C CNN
@@
 $EndComp
 $Comp
-L Earth #PWR021
+L Earth #PWR019
 U 1 1 58EDFF3B
 P 1350 5725
-F 0 "#PWR021" H 1350 5475 50  0001 C CNN
+F 0 "#PWR019" H 1350 5475 50  0001 C CNN
 F 1 "Earth" H 1350 5575 50  0001 C CNN
 F 2 "" H 1350 5725 50  0000 C CNN
@@
 NoConn ~ 2700 5525
 $Comp
-L Earth #PWR022
+L Earth #PWR020
 U 1 1 58EE190E
 P 700 4675
-F 0 "#PWR022" H 700 4425 50  0001 C CNN
+F 0 "#PWR020" H 700 4425 50  0001 C CNN
 F 1 "Earth" H 700 4525 50  0001 C CNN
 F 2 "" H 700 4675 50  0000 C CNN
@@
 $EndComp
 $Comp
-L Earth #PWR023
+L Earth #PWR021
 U 1 1 58EF3F4E
 P 4200 4675
-F 0 "#PWR023" H 4200 4425 50  0001 C CNN
+F 0 "#PWR021" H 4200 4425 50  0001 C CNN
 F 1 "Earth" H 4200 4525 50  0001 C CNN
 F 2 "" H 4200 4675 50  0000 C CNN
@@
 $EndComp
 $Comp
-L Earth #PWR024
+L Earth #PWR022
 U 1 1 58EF64C0
 P 675 2850
-F 0 "#PWR024" H 675 2600 50  0001 C CNN
+F 0 "#PWR022" H 675 2600 50  0001 C CNN
 F 1 "Earth" H 675 2700 50  0001 C CNN
 F 2 "" H 675 2850 50  0000 C CNN
@@
 $EndComp
 $Comp
-L Earth #PWR025
+L Earth #PWR023
 U 1 1 58F02228
 P 8475 3225
-F 0 "#PWR025" H 8475 2975 50  0001 C CNN
+F 0 "#PWR023" H 8475 2975 50  0001 C CNN
 F 1 "Earth" H 8475 3075 50  0001 C CNN
 F 2 "" H 8475 3225 50  0000 C CNN
@@
 3V3
 $Comp
-L Earth #PWR026
+L Earth #PWR024
 U 1 1 58F0BB40
 P 10200 1550
-F 0 "#PWR026" H 10200 1300 50  0001 C CNN
+F 0 "#PWR024" H 10200 1300 50  0001 C CNN
 F 1 "Earth" H 10200 1400 50  0001 C CNN
 F 2 "" H 10200 1550 50  0000 C CNN
@@
 RESET
 $Comp
-L Earth #PWR027
+L Earth #PWR025
 U 1 1 58EBC7CA
 P 8125 5025
-F 0 "#PWR027" H 8125 4775 50  0001 C CNN
+F 0 "#PWR025" H 8125 4775 50  0001 C CNN
 F 1 "Earth" H 8125 4875 50  0001 C CNN
 F 2 "" H 8125 5025 50  0000 C CNN
@@
 $EndComp
 $Comp
-L Earth #PWR028
+L Earth #PWR026
 U 1 1 58F62A82
 P 5325 5050
-F 0 "#PWR028" H 5325 4800 50  0001 C CNN
+F 0 "#PWR026" H 5325 4800 50  0001 C CNN
 F 1 "Earth" H 5325 4900 50  0001 C CNN
 F 2 "" H 5325 5050 50  0000 C CNN
@@
 VCC
 $Comp
-L Earth #PWR029
+L Earth #PWR027
 U 1 1 58F6D5C9
 P 5550 5800
-F 0 "#PWR029" H 5550 5550 50  0001 C CNN
+F 0 "#PWR027" H 5550 5550 50  0001 C CNN
 F 1 "Earth" H 5550 5650 50  0001 C CNN
 F 2 "" H 5550 5800 50  0000 C CNN
@@
 $EndComp
 $Comp
-L Earth #PWR030
+L Earth #PWR028
 U 1 1 58F73323
 P 4650 7525
-F 0 "#PWR030" H 4650 7275 50  0001 C CNN
+F 0 "#PWR028" H 4650 7275 50  0001 C CNN
 F 1 "Earth" H 4650 7375 50  0001 C CNN
 F 2 "" H 4650 7525 50  0000 C CNN
@@
 $EndComp
 Text GLabel 4900 7525 3    40   Input ~ 0
-VCC
+3V3
 $Comp
 L SW_SPST SW3
@@
 D8
 $Comp
-L Earth #PWR031
+L Earth #PWR029
 U 1 1 58F17F76
 P 5125 2825
-F 0 "#PWR031" H 5125 2575 50  0001 C CNN
+F 0 "#PWR029" H 5125 2575 50  0001 C CNN
 F 1 "Earth" H 5125 2675 50  0001 C CNN
 F 2 "" H 5125 2825 50  0000 C CNN
@@
 3V3
 $Comp
-L Earth #PWR032
+L Earth #PWR030
 U 1 1 58F1CD54
 P 6675 1575
-F 0 "#PWR032" H 6675 1325 50  0001 C CNN
+F 0 "#PWR030" H 6675 1325 50  0001 C CNN
 F 1 "Earth" H 6675 1425 50  0001 C CNN
 F 2 "" H 6675 1575 50  0000 C CNN
@@
 $EndComp
 $Comp
-L Earth #PWR033
+L Earth #PWR031
 U 1 1 58F1DBAD
 P 11000 1525
-F 0 "#PWR033" H 11000 1275 50  0001 C CNN
+F 0 "#PWR031" H 11000 1275 50  0001 C CNN
 F 1 "Earth" H 11000 1375 50  0001 C CNN
 F 2 "" H 11000 1525 50  0000 C CNN
@@
 $EndComp
 $Comp
-L Earth #PWR034
+L Earth #PWR032
 U 1 1 58F1F685
 P 7400 1575
-F 0 "#PWR034" H 7400 1325 50  0001 C CNN
+F 0 "#PWR032" H 7400 1325 50  0001 C CNN
 F 1 "Earth" H 7400 1425 50  0001 C CNN
 F 2 "" H 7400 1575 50  0000 C CNN
@@
 NoConn ~ 7275 2325
 $Comp
-L Earth #PWR035
+L Earth #PWR033
 U 1 1 58F25DBA
 P 5925 2275
-F 0 "#PWR035" H 5925 2025 50  0001 C CNN
+F 0 "#PWR033" H 5925 2025 50  0001 C CNN
 F 1 "Earth" H 5925 2125 50  0001 C CNN
 F 2 "" H 5925 2275 50  0000 C CNN
@@
 $EndComp
 $Comp
-L Earth #PWR036
+L Earth #PWR034
 U 1 1 58F25E94
 P 5925 2375
-F 0 "#PWR036" H 5925 2125 50  0001 C CNN
+F 0 "#PWR034" H 5925 2125 50  0001 C CNN
 F 1 "Earth" H 5925 2225 50  0001 C CNN
 F 2 "" H 5925 2375 50  0000 C CNN
@@
 $EndComp
 $Comp
-L Earth #PWR037
+L Earth #PWR035
 U 1 1 58F25F6E
 P 5925 2475
-F 0 "#PWR037" H 5925 2225 50  0001 C CNN
+F 0 "#PWR035" H 5925 2225 50  0001 C CNN
 F 1 "Earth" H 5925 2325 50  0001 C CNN
 F 2 "" H 5925 2475 50  0000 C CNN
@@
 $EndComp
 $Comp
-L Earth #PWR038
+L Earth #PWR036
 U 1 1 58F26048
 P 5925 2575
-F 0 "#PWR038" H 5925 2325 50  0001 C CNN
+F 0 "#PWR036" H 5925 2325 50  0001 C CNN
 F 1 "Earth" H 5925 2425 50  0001 C CNN
 F 2 "" H 5925 2575 50  0000 C CNN
@@
 $EndComp
 $Comp
-L PWR_FLAG #FLG039
+L PWR_FLAG #FLG037
 U 1 1 58F27EB0
 P 5375 5775
-F 0 "#FLG039" H 5375 5870 50  0001 C CNN
+F 0 "#FLG037" H 5375 5870 50  0001 C CNN
 F 1 "PWR_FLAG" V 5275 5875 50  0000 C CNN
 F 2 "" H 5375 5775 50  0000 C CNN
@@
 $EndComp
 $Comp
-L PWR_FLAG #FLG040
+L PWR_FLAG #FLG038
 U 1 1 58F2895D
 P 5375 5425
-F 0 "#FLG040" H 5375 5520 50  0001 C CNN
+F 0 "#FLG038" H 5375 5520 50  0001 C CNN
 F 1 "PWR_FLAG" V 5275 5525 50  0000 C CNN
 F 2 "" H 5375 5425 50  0000 C CNN
@@
 $EndComp
 $Comp
-L Earth #PWR041
+L Earth #PWR039
 U 1 1 58F362CD
 P 1175 4675
-F 0 "#PWR041" H 1175 4425 50  0001 C CNN
+F 0 "#PWR039" H 1175 4425 50  0001 C CNN
 F 1 "Earth" H 1175 4525 50  0001 C CNN
 F 2 "" H 1175 4675 50  0000 C CNN
@@
 Wire Wire Line
 	7525 4675 7525 4975
+Text GLabel 3200 6325 2    40   Input ~ 0
+VCC
+Text GLabel 2950 5925 2    40   Input ~ 0
+VCC
 $EndSCHEMATC
